Commit message: Add files via upload

File: ur_ros_cartesian_control/ur_ros_cartesian_control/urdf/mobile_manipulator.xacro (robot description, xacro)
@@ -6,4 +6,7 @@
         <xacro:property name="base_width" value="0.5" />
         <xacro:property name="manipulator_base_height" value="0.04" />
+        <material name="grey">
+            <color rgba="0.5 0.5 0.5 0.5" />
+        </material>
         <xacro:include filename="$(find ur_description)/urdf/inc/ur10_macro.xacro"/>
         <!-- *************************************************** -->
@@ -24,4 +27,5 @@
                     <box size="${base_length} ${base_width} ${base_height}"/>
                 </geometry>
+                <material name="grey"/>
             </collision>
             <!-- Inertial definitions are necessary for simulation -->
@@ -46,5 +50,5 @@
             <parent link="mobile_link"/>
             <child link="ur_base_link"/>
-            <origin xyz="0 0 ${base_height+manipulator_base_height/2}" rpy="0 0 3.141592"/>
+            <origin xyz="0.015 0.015 ${base_height+0.005+manipulator_base_height/2}" rpy="0 0 3.141592"/>
         </joint>
     </xacro:macro>
